File: HUB-SNMP/Hardware/HUB-SNMP.kicad_pcb (KiCad board)
At the start: 2 copper layers, 50.8 x 62.2 mm, 71 parts, among them J1 Conn_01x07_Male, T1 DTC114YKA, U1 ACPL-217-56AE, U2 TLV62569DBVT(SOT23-5), U3 ESP32-WROOM-32D-4MB, U4 LAN8710A-EZC(QFN32), U5 ACPL-217-56AE, U6 ACPL-217-56AE, U7 ACPL-217-56AE

Commit message: Proyecto de PCB en Kicad actualizados
-Se modifico el nombre del proyecto en kicad.
-Se generó el BOM actualizado.
-Se generó el pdf del esquematico actualizado.
-Se eliminaron archivos viejos innecesarios
Other:
- board text added: "SNMP Hub Casas Daiana Pregelj Jose Riveros Rubén Vieiro Alexis"
