File: HUB-SNMP/Hardware/HUB-SNMP.sch (KiCad schematic (older format))
At the start: 68 parts, among them J1 Conn_01x07_Male, T1 DTC114YKA, U1 ACPL-217-56AE, U2 TLV62569DBVT(SOT23-5), U3 ESP32-WROOM-32D-4MB, U4 LAN8710A-EZC(QFN32), U5 ACPL-217-56AE, U6 ACPL-217-56AE, U7 ACPL-217-56AE

Commit message: Proyecto de PCB en Kicad actualizados
-Se modifico el nombre del proyecto en kicad.
-Se generó el BOM actualizado.
-Se generó el pdf del esquematico actualizado.
-Se eliminaron archivos viejos innecesarios
Parts:
- C1, C11, C12, C13, C14, C15, C16, C17, C18, C19, C2, C20, C3, C4, C8, C9: symbol ESP32-GATEWAY_Rev_F:C -> HUB-SNMP-rescue:C-ESP32-GATEWAY_Rev_F
- FET1: symbol ESP32-GATEWAY_Rev_F:P-MOS+DIOD -> HUB-SNMP-rescue:P-MOS+DIOD-ESP32-GATEWAY_Rev_F
- FID2, FID3: symbol ESP32-GATEWAY_Rev_F:Fiducial -> HUB-SNMP-rescue:Fiducial-ESP32-GATEWAY_Rev_F
- GND1: symbol ESP32-GATEWAY_Rev_F:TESTPAD -> HUB-SNMP-rescue:TESTPAD-ESP32-GATEWAY_Rev_F
- L1, L2, L3: symbol ESP32-GATEWAY_Rev_F:L -> HUB-SNMP-rescue:L-ESP32-GATEWAY_Rev_F
- LAN1: symbol ESP32-GATEWAY_Rev_F:RJLBC-060TC1_GND -> HUB-SNMP-rescue:RJLBC-060TC1_GND-ESP32-GATEWAY_Rev_F
- MH1, MH2: symbol ESP32-GATEWAY_Rev_F:Mounting_hole_Shield_3.3mm -> HUB-SNMP-rescue:Mounting_hole_Shield_3.3mm-ESP32-GATEWAY_Rev_F
- PHY_RST1: symbol ESP32-GATEWAY_Rev_F:SJ -> HUB-SNMP-rescue:SJ-ESP32-GATEWAY_Rev_F
- R19, R20, R24, R25, R26, R27, R28, R29, R3, R31, R32, R33, R38, R39, R5, R54, R6: symbol ESP32-GATEWAY_Rev_F:R -> HUB-SNMP-rescue:R-ESP32-GATEWAY_Rev_F
- RM2, RM3: symbol ESP32-GATEWAY_Rev_F:RA1206_(4x0603)_4B8_Smashed -> HUB-SNMP-rescue:RA1206_(4x0603)_4B8_Smashed-ESP32-GATEWAY_Rev_F
- T1: symbol ESP32-GATEWAY_Rev_F:DTC114YKA -> HUB-SNMP-rescue:DTC114YKA-ESP32-GATEWAY_Rev_F
- U2: symbol ESP32-GATEWAY_Rev_F:SY8009AAAC(SOT23-5) -> HUB-SNMP-rescue:SY8009AAAC(SOT23-5)-ESP32-GATEWAY_Rev_F
- U3: symbol ESP32-GATEWAY_Rev_F:ESP-WROOM-32 -> HUB-SNMP-rescue:ESP-WROOM-32-ESP32-GATEWAY_Rev_F
- U4: symbol ESP32-GATEWAY_Rev_F:LAN8710A-EZC(QFN32) -> HUB-SNMP-rescue:LAN8710A-EZC(QFN32)-ESP32-GATEWAY_Rev_F
- USB-UART2: symbol ESP32-GATEWAY_Rev_F-rescue:USB_B_Micro-Connector -> HUB-SNMP-rescue:USB_B_Micro-Connector-ESP32-GATEWAY_Rev_F-rescue
Connections:
- net labels added: GPIO16\DOOR4
- net labels removed: GPIO16
Other:
- moved on the sheet: FID2, FID3
